File: hardware/simpanel/simpanel.kicad_pcb (KiCad board)
At the start: 2 copper layers, 391.2 x 137.2 mm, 46 parts, among them J1 Power, J2 Conn_02x12_Top_Bottom, U1 AS1130-BSST, U2 AS1130-BSST, U3 4504, U4 4504, U5 4504, U6 4504

Commit message: Rev C
Parts:
- removed DS1, DS10, DS11, DS12, DS13, DS14, DS15, DS16, DS2, DS3, DS4, DS5, DS6, DS7, DS8, DS9: LTP-587HR, LTP-587HR:DIPS1270W50P254L2500H975Q18N
- removed H5, H6: MountingHole_Pad, MountingHole:MountingHole_3.7mm_Pad_Via
- removed S2, S3, S4, S5, S6, S7: B3J-2100, B3J-2100:B3J2100
- removed SHIELD1: VAL**, arduino_shields:ARDUINO MEGA SHIELD
- removed the U3 at (229.9, 120.7)
- added C1: 47µf, Capacitor_SMD:C_Elec_4x5.4, F.Cu at (125.7, 99.7)
- added C2: 100nf, Capacitor_SMD:C_0603_1608Metric, F.Cu at (123.2, 109.2)
- added C3: 1µf, Capacitor_SMD:C_0603_1608Metric, F.Cu at (168.9, 85.7)
- added C4: 22pf, Capacitor_SMD:C_0603_1608Metric, F.Cu at (179.7, 107.3)
- added C5: 22pf, Capacitor_SMD:C_0603_1608Metric, F.Cu at (177.8, 107.3)
- added C6: 100nf, Capacitor_SMD:C_0603_1608Metric, F.Cu at (156.2, 112.4)
- added FB1: BLM21, Resistor_SMD:R_0603_1608Metric, F.Cu at (141.6, 111.1)
- added J3: ISP, Connector_PinHeader_2.54mm:PinHeader_2x03_P2.54mm_Vertical, F.Cu at (165.7, 120.7)
- added R1: 22, Resistor_SMD:R_0603_1608Metric, F.Cu at (134.0, 104.1)
- added R2: 22, Resistor_SMD:R_0603_1608Metric, F.Cu at (132.1, 104.1)
- added R3: CG0603MLC-05E, Resistor_SMD:R_0603_1608Metric, F.Cu at (127.6, 111.1)
- added R4: CG0603MLC-05E, Resistor_SMD:R_0603_1608Metric, F.Cu at (139.1, 111.1)
- added R5: 10k, Resistor_SMD:R_0603_1608Metric, F.Cu at (163.2, 95.9)
- added SW12: SW_Push, XKB5858-W-C:XKB5858WC, F.Cu at (156.8, 115.6)
- added SW2: B3J-2100, simpanel:B3J2100, F.Cu at (89.5, 104.1)
- added SW3: B3J-2100, simpanel:B3J2100, F.Cu at (89.5, 76.2)
- added SW4: B3J-2100, simpanel:B3J2100, F.Cu at (89.5, 54.0)
- added SW5: B3J-2100, simpanel:B3J2100, F.Cu at (112.4, 104.1)
- added SW6: B3J-2100, simpanel:B3J2100, F.Cu at (151.8, 104.1)
- added SW7: B3J-2100, simpanel:B3J2100, F.Cu at (202.6, 104.1)
- added U1: AT90USB1286-AU, Package_QFP:TQFP-64_14x14mm_P0.8mm, F.Cu at (179.7, 88.3)
- added U7: SLR0363DWC1BD, simpanel:SLR0363DWC1BD, F.Cu at (142.9, 42.5)
- added U8: SLR0363DWC1BD, simpanel:SLR0363DWC1BD, F.Cu at (114.9, 42.5)
- added U9: SLR0363DWC1BD, simpanel:SLR0363DWC1BD, F.Cu at (69.2, 42.5)
- added Y1: 16MHz, Crystal:Crystal_SMD_HC49-SD, F.Cu at (178.9, 102.9)
- ENC1, ENC2, ENC3, ENC4: footprint pecr11:Bourns-PEC11R-4220F-S0024-0-0-0 -> simpanel:PEC11R
- J1: value Power -> U-F-M5DW-Y-2; footprint Connector_Molex:Molex_Micro-Fit_3.0_43650-0300_1x03_P3.00mm_Horizontal -> digikey-kicad-library-master:USB_Micro_B_Female_10118194-0001LF; moved to F.Cu
- J2: value Conn_02x12_Top_Bottom -> Conn_2Rows-21Pins; footprint Connector_Molex:Molex_Micro-Fit_3.0_43045-2400_2x12_P3.00mm_Horizontal -> Connector_PinHeader_2.54mm:PinHeader_2x11_P2.54mm_Vertical
- SW1: renamed from S1; footprint B3J-2100:B3J2100 -> simpanel:B3J2100
- SW10: renamed from S10; footprint B3J-2100:B3J2100 -> simpanel:B3J2100
- SW11: renamed from S11; footprint B3J-2100:B3J2100 -> simpanel:B3J2100
- SW8: renamed from S8; footprint B3J-2100:B3J2100 -> simpanel:B3J2100
- SW9: renamed from S9; footprint B3J-2100:B3J2100 -> simpanel:B3J2100
- U4, U5, U6: value 4504 -> SLR0363DWC1BD; footprint Package_DIP:DIP-16_W7.62mm -> simpanel:SLR0363DWC1BD
- moved SW10 334.0 mm to (44.5, 76.2)
- moved J1 177.2 mm to (133.3, 108.6)
- moved U6 154.0 mm to (165.7, 42.5), turned to 0 degrees
- moved SW8 145.4 mm to (236.9, 104.1)
- moved SW9 144.7 mm to (236.9, 79.4)
- moved SW11 141.6 mm to (236.9, 54.0)
- moved ENC4 122.8 mm to (205.1, 67.3)
- moved U5 113.2 mm to (193.7, 42.5), turned to 0 degrees
- moved U2 95.2 mm to (179.7, 60.3)
- moved U4 86.1 mm to (216.5, 42.5), turned to 0 degrees
- moved ENC3 68.2 mm to (154.3, 67.3)
- moved J2 62.5 mm to (196.2, 118.1), turned to 270 degrees
- moved H4 43.9 mm to (236.9, 118.1)
- moved H3 41.6 mm to (225.4, 57.1)
- moved H2 34.3 mm to (50.8, 118.1)
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- renumbered U1 to U2, U2 to U3
Connections:
- net /RST renamed /PC7
- J1 pad 1: GND -> VCC
- J1 pad 2: VDD -> /UD-
- J1 pad 3: VCC -> /UD+
- J2 pad 1: Net-(J2-Pad1) -> /PF1
- J2 pad 10: Net-(J2-Pad10) -> /PF6
- J2 pad 11: Net-(J2-Pad11) -> /PE4
- J2 pad 12: VCC -> /PF7
- J2 pad 13: Net-(J2-Pad13) -> /PE3
- J2 pad 14: Net-(J2-Pad14) -> /PD7
- J2 pad 15: Net-(J2-Pad15) -> /PE2
- J2 pad 16: Net-(J2-Pad16) -> /PD6
- J2 pad 17: Net-(J2-Pad17) -> /PE1
- J2 pad 18: Net-(J2-Pad18) -> /PD5
- J2 pad 19: Net-(J2-Pad19) -> /PE0
- J2 pad 2: Net-(J2-Pad2) -> /PF2
- J2 pad 20: Net-(J2-Pad20) -> /PD4
- J2 pad 21: Net-(J2-Pad21) -> GND
- J2 pad 22: Net-(J2-Pad22) -> (no net)
- J2 pad 3: Net-(J2-Pad3) -> /PF0
- J2 pad 4: Net-(J2-Pad4) -> /PF3
- J2 pad 5: Net-(J2-Pad5) -> /PE7
- J2 pad 6: Net-(J2-Pad6) -> /PF4
- J2 pad 7: Net-(J2-Pad7) -> /PE6
- J2 pad 8: Net-(J2-Pad8) -> /PF5
- J2 pad 9: Net-(J2-Pad9) -> /PE5
- SW1 pad 3: /SW1 -> /PC6
- SW1 pad 4: Net-(S1-Pad4) -> (no net)
- SW1 pad A1: /U2CS4 -> /CSB0
- SW1 pad K1: /U2CS0 -> /CSB11
- SW10 pad 3: /SW10 -> /PB5
- SW10 pad 4: Net-(S10-Pad4) -> (no net)
- SW10 pad A1: /U2CS4 -> /CSB9
- SW10 pad K1: /U2CS10 -> /CSB11
- SW11 pad 3: /SW11 -> /PB4
- SW11 pad 4: Net-(S11-Pad4) -> (no net)
- SW11 pad A1: /U2CS4 -> /CSB10
- SW11 pad K1: /U2CS11 -> /CSB11
- SW8 pad 3: /SW8 -> /PB7
- SW8 pad 4: Net-(S8-Pad4) -> (no net)
- SW8 pad A1: /U2CS4 -> /CSB7
- SW8 pad K1: /U2CS8 -> /CSB11
- SW9 pad 3: /SW9 -> /PB6
- SW9 pad 4: Net-(S9-Pad4) -> (no net)
- SW9 pad A1: /U2CS4 -> /CSB8
- SW9 pad K1: /U2CS9 -> /CSB11
- U2 pad 10: VDD -> VCC
- U2 pad 11: /U1IRQ -> /IRQA
- U2 pad 17: Net-(U1-Pad17) -> (no net)
- U2 pad 18: VDD -> VCC
- U2 pad 19: VDD -> VCC
- U2 pad 2: /U1CS6 -> /CSA6
- U2 pad 20: /U1CS5 -> /CSA5
- U2 pad 21: /U1CS4 -> /CSA4
- U2 pad 23: /U1CS2 -> /CSA2
- U2 pad 24: /U1CS3 -> /CSA3
- U2 pad 25: /U1CS0 -> /CSA0
- U2 pad 26: Net-(U1-Pad26) -> VCC
- U2 pad 27: /U1CS1 -> /CSA1
- U2 pad 3: VDD -> VCC
- U2 pad 4: /U1CS7 -> /CSA7
- U2 pad 5: /U1CS8 -> /CSA8
- U2 pad 6: /U1CS9 -> /CSA9
- U2 pad 7: Net-(U1-Pad7) -> GND
- U2 pad 8: /U1CS11 -> /CSA11
- U2 pad 9: /U1CS10 -> /CSA10
- U3 pad 10: VDD -> VCC
- U3 pad 11: /U2IRQ -> /IRQB
- U3 pad 18: VDD -> VCC
- U3 pad 19: VDD -> VCC
- U3 pad 2: /U2CS6 -> /CSB6
- U3 pad 20: /U2CS5 -> /CSB5
- U3 pad 21: /U2CS4 -> /CSB4
- U3 pad 22: Net-(U2-Pad22) -> GND
- U3 pad 23: /U2CS2 -> /CSB2
- U3 pad 24: /U2CS3 -> /CSB3
- U3 pad 25: /U2CS0 -> /CSB0
- U3 pad 26: Net-(U2-Pad26) -> VCC
- U3 pad 27: /U2CS1 -> /CSB1
- U3 pad 3: VDD -> VCC
- U3 pad 4: /U2CS7 -> /CSB7
- U3 pad 5: /U2CS8 -> /CSB8
- U3 pad 6: /U2CS9 -> /CSB9
- U3 pad 8: /U2CS11 -> /CSB11
- U3 pad 9: /U2CS10 -> /CSB10
- U4 pad 1: VCC -> /CSA7
- U4 pad 10: Net-(SHIELD1-Pad41) -> /CSA8
- U4 pad 11: Net-(J2-Pad16) -> /CSA3
- U4 pad 12: Net-(SHIELD1-Pad40) -> /CSA0
- U4 pad 2: Net-(SHIELD1-Pad44) -> /CSA6
- U4 pad 3: Net-(J2-Pad18) -> /CSA10
- U4 pad 4: Net-(SHIELD1-Pad43) -> /CSA5
- U4 pad 5: Net-(J2-Pad5) -> /CSA9
- U4 pad 6: Net-(SHIELD1-Pad42) -> (no net)
- U4 pad 7: Net-(J2-Pad6) -> /CSA4
- U4 pad 8: GND -> /CSA2
- U4 pad 9: Net-(J2-Pad17) -> /CSA1
- U5 pad 1: VCC -> /CSA7
- U5 pad 10: Net-(SHIELD1-Pad47) -> /CSA8
- U5 pad 11: Net-(J2-Pad19) -> /CSA0
- U5 pad 12: Net-(SHIELD1-Pad46) -> /CSA3
- U5 pad 2: Net-(SHIELD1-Pad51) -> /CSA6
- U5 pad 3: Net-(J2-Pad21) -> /CSA10
- U5 pad 4: Net-(SHIELD1-Pad49) -> /CSA2
- U5 pad 5: Net-(J2-Pad8) -> /CSA9
- U5 pad 6: Net-(SHIELD1-Pad48) -> (no net)
- U5 pad 7: Net-(J2-Pad9) -> /CSA1
- U5 pad 8: GND -> /CSA5
- U5 pad 9: Net-(J2-Pad20) -> /CSA4
- U6 pad 1: VCC -> /CSA4
- U6 pad 10: Net-(SHIELD1-Pad8) -> /CSA5
- U6 pad 11: Net-(J2-Pad22) -> /CSA0
- U6 pad 12: Net-(SHIELD1-Pad9) -> /CSA6
- U6 pad 2: Net-(U6-Pad2) -> /CSA3
- U6 pad 3: Net-(U6-Pad3) -> /CSA10
- U6 pad 4: Net-(U6-Pad4) -> /CSA2
- U6 pad 5: Net-(U6-Pad5) -> /CSA9
- U6 pad 6: Net-(SHIELD1-Pad7) -> (no net)
- U6 pad 7: Net-(J2-Pad11) -> /CSA1
- U6 pad 8: GND -> /CSA8
- U6 pad 9: Net-(J2-Pad23) -> /CSA7
Routing:
- net /U2CS4: track 640.2 -> 0.00 mm, vias 2 -> 0
- net VDD: track 588.1 -> 0.00 mm, vias 4 -> 0
- net /U2CS7: track 485.4 -> 0.00 mm, vias 2 -> 0
- net /U2CS8: track 482.9 -> 0.00 mm, vias 2 -> 0
- net /U2CS9: track 475.7 -> 0.00 mm, vias 2 -> 0
- net /CSB11: track 0.00 -> 452.0 mm, vias 0 -> 3
- net /SW11: track 443.8 -> 0.00 mm, vias 1 -> 0
- net /SW10: track 420.2 -> 0.00 mm, vias 1 -> 0
- net /U2CS11: track 406.9 -> 0.00 mm, vias 2 -> 0
- net GND: track 1288.4 -> 900.5 mm, vias 5 -> 2
- net /SW9: track 385.9 -> 0.00 mm, vias 1 -> 0
- net /U2CS10: track 377.2 -> 0.00 mm, vias 2 -> 0
- net /SW8: track 358.2 -> 0.00 mm, vias 1 -> 0
- net /U1CS5: track 322.0 -> 0.00 mm, vias 6 -> 0
- net /U1CS11: track 315.0 -> 0.00 mm, vias 4 -> 0
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- added copper zone on B.Cu, net GND
Other:
- board size 391.2 x 137.2 mm -> 206.4 x 99.1 mm
- net class Default: via_dia 0.7 -> 0.6; via_drill 0.35 -> 0.3
- net class Supply: trace_width 0.45 -> 0.5
- board text added: "2021 © Marc A. Pelletier"
- board text added: "SIMPANEL rev. C 20210716-2"
- board text removed: "- +12V"
- board text removed: "- +5V"
- board text removed: "- GND"
- board text removed: "2020 © Marc A. Pelletier"
- board text removed: "JLCJLCJLCJLC"
- board text removed: "SIMPANEL rev. A 20201210-2"
